File: EAGLE/projects/New_Project_2/b_SI_Boost.brd (EAGLE design)
At the start: 196.8 x 83.5 mm, 28 parts, among them J1 66.9040-22, J10 66.9040-22, J11 66.9040-22, J12 66.9040-22, J13 66.9040-22, J14 66.9040-22, J15 66.9040-22, J16 66.9040-22, J2 66.9040-22, J3 66.9040-22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

Commit message: some corrections in eagle
Parts:
- removed J5: 66.9040-22, SamacSys_Parts:66904022
Connections:
- removed net N$7: J5.1, J5.2, J5.3, J5.4, J5.5, Q2.1
- new net N$9: Q2.1
Routing:
- net N$7: track 32.0 -> 0.00 mm
Changed lines of the file:
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@@
 <attribute name="VALUE" x="200.66" y="8.89" size="1.27" layer="27" rot="R270" align="center"/>
-</element>
-<element name="J5" library="SamacSys_Parts" package="66904022" value="66.9040-22" x="162.56" y="11.43" smashed="yes" rot="R180">
-<attribute name="ALLIED_NUMBER" value="70749834" x="81.28" y="90.17" size="1.778" layer="27" rot="R180" display="off"/>
-<attribute name="ALLIED_PRICE-STOCK" value="https://www.alliedelec.com/staubli-66-9040-22/70749834/" x="81.28" y="90.17" size="1.778" layer="27" rot="R180" display="off"/>
-<attribute name="ARROW_PART_NUMBER" value="66.9040-22" x="81.28" y="90.17" size="1.778" layer="27" rot="R180" display="off"/>
-<attribute name="ARROW_PRICE-STOCK" value="" x="81.28" y="90.17" size="1.778" layer="27" rot="R180" display="off"/>
-<attribute name="DESCRIPTION" value="STAUBLI - 66.9040-22 - SOCKET, PCB, 4MM, R/A, RED" x="81.28" y="90.17" size="1.778" layer="27" rot="R180" display="off"/>
-<attribute name="HEIGHT" value="11mm" x="81.28" y="90.17" size="1.778" layer="27" rot="R180" display="off"/>
-<attribute name="MANUFACTURER_NAME" value="STAUBLI" x="81.28" y="90.17" size="1.778" layer="27" rot="R180" display="off"/>
-<attribute name="MANUFACTURER_PART_NUMBER" value="66.9040-22" x="81.28" y="90.17" size="1.778" layer="27" rot="R180" display="off"/>
-<attribute name="NAME" x="162.56" y="6.35" size="1.27" layer="25" rot="R180" align="center"/>
-<attribute name="RS_PART_NUMBER" value="" x="81.28" y="90.17" size="1.778" layer="27" rot="R180" display="off"/>
-<attribute name="RS_PRICE-STOCK" value="" x="81.28" y="90.17" size="1.778" layer="27" rot="R180" display="off"/>
-<attribute name="VALUE" x="162.56" y="8.89" size="1.27" layer="27" rot="R180" align="center"/>
 </element>
 <element name="J6" library="SamacSys_Parts" package="66904022" value="66.9040-22" x="172.72" y="85.09" smashed="yes">
@@
 <wire x1="151.13" y1="62.23" x2="160.02" y2="70.43" width="0" layer="19" extent="1-1"/>
 </signal>
-<signal name="N$7">
-<contactref element="Q2" pad="1"/>
-<contactref element="J5" pad="2"/>
-<contactref element="J5" pad="4"/>
-<contactref element="J5" pad="5"/>
-<contactref element="J5" pad="1"/>
-<contactref element="J5" pad="3"/>
-<wire x1="157.48" y1="26.09" x2="158.76" y2="26.09" width="2.54" layer="1"/>
-<wire x1="158.76" y1="26.09" x2="162.56" y2="22.29" width="2.54" layer="1"/>
-<wire x1="162.56" y1="22.29" x2="166.36" y2="26.09" width="2.54" layer="1"/>
-<wire x1="166.36" y1="26.09" x2="167.64" y2="26.09" width="2.54" layer="1"/>
-<wire x1="167.64" y1="15.93" x2="167.64" y2="17.21" width="2.54" layer="1"/>
-<wire x1="167.64" y1="17.21" x2="162.56" y2="22.29" width="2.54" layer="1"/>
-<wire x1="162.56" y1="22.29" x2="157.48" y2="17.21" width="2.54" layer="1"/>
-<wire x1="157.48" y1="17.21" x2="157.48" y2="15.93" width="2.54" layer="1"/>
-<wire x1="163.83" y1="23.56" x2="162.56" y2="22.29" width="2.54" layer="1"/>
-<wire x1="166.36" y1="26.09" x2="163.83" y2="60.96" width="0" layer="19" extent="1-1"/>
-</signal>
 <signal name="N$8">
 <contactref element="D8" pad="2"/>
@@
 <wire x1="168.92" y1="70.43" x2="169.27" y2="60.96" width="0" layer="19" extent="1-1"/>
 </signal>
+<signal name="N$9">
+<contactref element="Q2" pad="1"/>
+</signal>
 </signals>
