File: EAGLE/projects/New_Project_2/b_SI_Boost.sch (EAGLE design)
At the start: 23 parts, among them J1 66.9040-22, J10 66.9040-22, J11 66.9040-22, J12 66.9040-22, J13 66.9040-22, J14 66.9040-22, J15 66.9040-22, J16 66.9040-22, J2 66.9040-22, J3 66.9040-22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

Commit message: some corrections in eagle
Parts:
- removed J5: 66.9040-22, SamacSys_Parts:66.9040-22
Connections:
- removed net N$7: J5.1, J5.2, J5.3, J5.4, J5.5, Q2.G
- new net N$9: Q2.G
Changed lines of the file:
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@@
 <part name="J8" library="SamacSys_Parts" deviceset="66.9040-22" device=""/>
 <part name="J10" library="SamacSys_Parts" deviceset="66.9040-22" device=""/>
-<part name="J5" library="SamacSys_Parts" deviceset="66.9040-22" device=""/>
 <part name="J2" library="SamacSys_Parts" deviceset="66.9040-22" device=""/>
 <part name="J11" library="SamacSys_Parts" deviceset="66.9040-22" device=""/>
@@
 <attribute name="NAME" x="-16.51" y="-10.16" size="1.778" layer="95" align="center-left"/>
 <attribute name="VALUE" x="-16.51" y="-12.7" size="1.778" layer="96" align="center-left"/>
-</instance>
-<instance part="J5" gate="G$1" x="78.74" y="-40.64" smashed="yes">
-<attribute name="NAME" x="95.25" y="-33.02" size="1.778" layer="95" align="center-left"/>
-<attribute name="VALUE" x="95.25" y="-35.56" size="1.778" layer="96" align="center-left"/>
 </instance>
 <instance part="J2" gate="G$1" x="50.8" y="33.02" smashed="yes" rot="R270">
@@
 </segment>
 </net>
-<net name="N$7" class="0">
-<segment>
-<pinref part="Q2" gate="G$1" pin="G"/>
-<pinref part="J5" gate="G$1" pin="2"/>
-<wire x1="99.06" y1="-40.64" x2="99.06" y2="-38.1" width="0.1524" layer="91"/>
-<pinref part="J5" gate="G$1" pin="4"/>
-<wire x1="99.06" y1="-43.18" x2="99.06" y2="-40.64" width="0.1524" layer="91"/>
-<junction x="99.06" y="-40.64"/>
-<junction x="99.06" y="-43.18"/>
-<pinref part="J5" gate="G$1" pin="5"/>
-<pinref part="J5" gate="G$1" pin="1"/>
-<wire x1="78.74" y1="-40.64" x2="78.74" y2="-43.18" width="0.1524" layer="91"/>
-<pinref part="J5" gate="G$1" pin="3"/>
-<junction x="78.74" y="-43.18"/>
-<wire x1="78.74" y1="-43.18" x2="78.74" y2="-45.72" width="0.1524" layer="91"/>
-<wire x1="99.06" y1="-38.1" x2="78.74" y2="-38.1" width="0.1524" layer="91"/>
-<wire x1="78.74" y1="-38.1" x2="78.74" y2="-40.64" width="0.1524" layer="91"/>
-<junction x="78.74" y="-40.64"/>
-<junction x="99.06" y="-38.1"/>
-</segment>
-</net>
 <net name="N$8" class="0">
 <segment>
@@
 </segment>
 </net>
+<net name="N$9" class="0">
+<segment>
+<pinref part="Q2" gate="G$1" pin="G"/>
+<wire x1="99.06" y1="-43.18" x2="99.06" y2="-38.1" width="0.1524" layer="91"/>
+</segment>
+</net>
