File: EAGLE/projects/New_Project_2/3level_2NX_interleaved_boost_converter.sch (EAGLE design)
At the start: 32 parts, among them J1 26-60-4050, J3 66.9040-22, J4 66.9040-22, J5 66.9040-22, J6 66.9040-22, J7 26-60-4050, Q1 C2M0160120D, Q2 C2M0160120D

Commit message: 3 stage pcb done
want to look over it tomorrow, can probably be sent, but am not sure about the bobbin spacing
Parts:
- removed J3, J4, J5, J6: 66.9040-22, SamacSys_Parts:66.9040-22
- removed L1, L2: CTX100-10-52LPR, SamacSys_Parts:CTX100-10-52LPR
- added H1, H10, H11, H12, H13, H14, H15, H16, H17, H18, H2, H3, H4, H5, H6, H7, H8, H9: MOUNT-PAD-ROUND5.0, holes:MOUNT-PAD-ROUND5.0
- added KK1, KK10, KK11, KK12, KK13, KK2, KK3, KK4, KK5, KK6, KK7, KK8, KK9: SK104-PAD, heatsink:SK104-PAD
- added U$1, U$2: JELL, placeholders:JELL
- C1, C10, C11, C2, C3, C4, C5, C6, C7, C8, C9: value B32774D4505K000 -> SANJEECAP; device SamacSys_Parts:B32774D4505K000 -> placeholders:SANJEECAP
Connections:
- net GND: now also H11.MOUNT, H8.MOUNT; no longer J6.1, J6.2, J6.3, J6.4, J6.5
- net N$1: now also H15.MOUNT
- net N$10: now also H10.MOUNT
- net N$11: now also H13.MOUNT
- net N$17: now also H17.MOUNT
- net N$18: now also H9.MOUNT
- net N$2: now also H4.MOUNT; no longer L1.2
- net N$3: now also H12.MOUNT
- net N$4: now also H14.MOUNT
- net N$5: now also H2.MOUNT; no longer L2.2
- net N$6: now also H5.MOUNT; no longer J3.1, J3.2, J3.3, J3.4, J3.5
- net N$7: now also H18.MOUNT
- net N$8: now also H6.MOUNT; no longer J4.1, J4.2, J4.3, J4.4, J4.5
- net N$9: now also H16.MOUNT
- net VCC: now also H1.MOUNT, H3.MOUNT, H7.MOUNT; no longer J5.1, J5.2, J5.3, J5.4, J5.5, L1.1, L2.1
