File: EAGLE/projects/New_Project_2/3level_2NX_interleaved_boost_converter.brd (EAGLE design)
At the start: 180 x 280 mm, 32 parts, among them J1 26-60-4050, J3 66.9040-22, J4 66.9040-22, J5 66.9040-22, J6 66.9040-22, J7 26-60-4050, Q1 C2M0160120D, Q2 C2M0160120D

Commit message: 3 stage pcb done
want to look over it tomorrow, can probably be sent, but am not sure about the bobbin spacing
Parts:
- removed J3, J4, J5, J6: 66.9040-22, SamacSys_Parts:66904022
- removed L1, L2: CTX100-10-52LPR, SamacSys_Parts:CTX1001052LPR
- added H1, H10, H11, H12, H13, H14, H15, H16, H17, H18, H2, H3, H4, H5, H6, H7, H8, H9: MOUNT-PAD-ROUND5.0, holes:5,0-PAD
- added KK1, KK10, KK11, KK12, KK13, KK2, KK3, KK4, KK5, KK6, KK7, KK8, KK9: SK104-PAD, heatsink:SK104-PAD
- added U$1, U$2: JELL, placeholders:BOBBIN
- C1, C10, C11, C2, C3, C4, C5, C6, C7, C8, C9: value B32774D4505K000 -> SANJEECAP; device SamacSys_Parts:B32774D4505K000 -> placeholders:ECA2WHG2R2
- moved Q2 35.7 mm to (47.0, 116.0), turned to 90 degrees
- moved J7 31.5 mm to (35.5, 121.0), turned to 270 degrees
- moved C2 24.3 mm to (50.0, 100.0), turned to 270 degrees
- moved C3 23.8 mm to (97.0, 175.0), turned to 270 degrees
- moved D11 23.5 mm to (78.5, 127.0)
- moved C4 22.9 mm to (50.0, 65.0), turned to 270 degrees
- moved C11 22.8 mm to (50.0, 30.0), turned to 270 degrees
- moved D7 21.4 mm to (62.4, 25.5)
- moved C6 20.5 mm to (97.0, 210.0), turned to 270 degrees
- moved C8 20.1 mm to (50.0, 220.0), turned to 270 degrees
- moved C9 19.7 mm to (97.0, 245.0), turned to 270 degrees
- moved D5 19.6 mm to (62.5, 64.0)
- moved C1 19.4 mm to (50.0, 185.0), turned to 270 degrees
- moved D9 19.0 mm to (62.5, 265.0)
- moved D6 18.9 mm to (62.5, 227.0)
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Connections:
- net GND: now also C10.PLUS, C3.MINUS, H11.B5, H8.B5; no longer C10.2, C3.1, J6.1, J6.2, J6.3, J6.4, J6.5
- net N$1: now also C1.PLUS, C8.MINUS, H15.B5; no longer C1.2, C8.1
- net N$10: now also C10.MINUS, C5.PLUS, H10.B5; no longer C10.1, C5.2
- net N$11: now also C6.PLUS, C9.MINUS, H13.B5; no longer C6.2, C9.1
- net N$17: now also C11.PLUS, C4.MINUS, H17.B5; no longer C11.2, C4.1
- net N$18: now also C5.MINUS, C7.PLUS, H9.B5; no longer C5.1, C7.2
- net N$2: now also C1.MINUS, H4.B5; no longer C1.1, L1.2
- net N$3: now also C3.PLUS, C6.MINUS, H12.B5; no longer C3.2, C6.1
- net N$4: now also C8.PLUS, H14.B5; no longer C8.2
- net N$5: now also C2.PLUS, H2.B5; no longer C2.2, L2.2
- net N$6: now also C9.PLUS, H5.B5; no longer C9.2, J3.1, J3.2, J3.3, J3.4, J3.5
- net N$7: now also C11.MINUS, H18.B5; no longer C11.1
- net N$8: now also C7.MINUS, H6.B5; no longer C7.1, J4.1, J4.2, J4.3, J4.4, J4.5
- net N$9: now also C2.MINUS, C4.PLUS, H16.B5; no longer C2.1, C4.2
- net VCC: now also H1.B5, H3.B5, H7.B5; no longer J5.1, J5.2, J5.3, J5.4, J5.5, L1.1, L2.1
Routing:
- net N$2: track 0.00 -> 71.1 mm
- net N$5: track 0.00 -> 59.5 mm
- net N$13: track 0.00 -> 20.0 mm
- net N$12: track 0.00 -> 19.8 mm
- net GND: track 0.00 -> 9.78 mm
- added copper zone on layer 16, net GND
- added copper zone on layer 16, net N$1
- added copper zone on layer 16, net N$10
- added copper zone on layer 16, net N$11
- added copper zone on layer 16, net N$17
- added copper zone on layer 16, net N$18
- added copper zone on layer 16, net N$3
- added copper zone on layer 16, net N$4
- added copper zone on layer 16, net N$6
- added copper zone on layer 16, net N$7
- added copper zone on layer 16, net N$8
- added copper zone on layer 16, net N$9
- added copper zone on layer 16, net VCC
Other:
- board text added: "AAU"
- board text added: "Lbot"
- board text added: "Ltop"
- board text added: "P5 project by ED5-3-F18: Daniel Busemann Ilian Haralampiev Ivan Kulin Simon Thies"
- board text added: "Vin"

Commit message: GERBER
 board should have the correct size now
Parts:
- moved U$2 1.50 mm to (2.10, 73.2)
Other:
- board size 180 x 280 mm -> 105 x 280 mm
Changed lines of the file:
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@@
 <board>
 <plain>
-<wire x1="0" y1="0" x2="180" y2="0" width="0" layer="20" locked="yes"/>
-<wire x1="180" y1="0" x2="180" y2="280" width="0" layer="20"/>
-<wire x1="180" y1="280" x2="0" y2="280" width="0" layer="20"/>
+<wire x1="0" y1="0" x2="105" y2="0" width="0" layer="20"/>
+<wire x1="105" y1="0" x2="105" y2="280" width="0" layer="20"/>
+<wire x1="105" y1="280" x2="0" y2="280" width="0" layer="20"/>
 <wire x1="0" y1="280" x2="0" y2="0" width="0" layer="20"/>
 <text x="12" y="140" size="6.4516" layer="25" rot="R90" align="bottom-center">Vin</text>
@@
 <attribute name="NAME" x="-0.319665625" y="179.892" size="1.27" layer="25" rot="R90"/>
 </element>
-<element name="U$2" library="placeholders" package="BOBBIN" value="JELL" x="3" y="72" smashed="yes" rot="R90">
-<attribute name="NAME" x="3.680334375" y="75.892" size="1.27" layer="25" rot="R90"/>
+<element name="U$2" library="placeholders" package="BOBBIN" value="JELL" x="2.1" y="73.2" smashed="yes" rot="R90">
+<attribute name="NAME" x="2.780334375" y="77.092" size="1.27" layer="25" rot="R90"/>
 </element>
 <element name="H1" library="holes" library_urn="urn:adsk.eagle:library:237" package="5,0-PAD" package3d_urn="urn:adsk.eagle:package:14288/1" value="MOUNT-PAD-ROUND5.0" x="18" y="150" smashed="yes"/>
@@
 packages will not be understood (or retained) with this version.
 </note>
-<note version="8.5" severity="warning">
-Since Version 8.5, EAGLE supports locking for holes, vias, wires and polygons.
-The locking property on all objects of these types will not be understood in this version.
-</note>
 </compatibility>
